File: ultrasonic_anemometer.kicad_pcb (KiCad board)
At the start: 2 copper layers, 110.5 x 39.4 mm, 51 parts, among them J1 Conn_01x04, Q1 BC857, Q2 BC857, U1 LM324, U2 EM78P153S, U3 MAX232A, Y1 27MHz

Commit message: Actual updated kicad files
(forgot to save my project before committing)
Other:
- board text added: "V0.1"
Changed lines of the file:
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@@
     (links 91)
     (no_connects 0)
-    (area 96.444999 82.655 207.085001 125.397619)
+    (area 96.444999 79.6954 207.085001 125.397619)
     (thickness 1.6)
-    (drawings 9)
+    (drawings 10)
     (tracks 588)
     (zones 0)
@@
     (tags "mounting hole 3mm no annular")
     (attr virtual)
-    (fp_text reference REF** (at 0 -4) (layer F.SilkS)
+    (fp_text reference REF** (at 0 -4) (layer F.SilkS) hide
       (effects (font (size 1 1) (thickness 0.15)))
     )
@@
     (tags "capacitor 0603")
     (attr smd)
-    (fp_text reference C15 (at 0 -1.25 90) (layer F.SilkS)
+    (fp_text reference C15 (at 0 -1.25 90) (layer F.SilkS) hide
       (effects (font (size 1 1) (thickness 0.15)))
     )
@@
       (effects (font (size 1 1) (thickness 0.15)))
     )
-    (fp_text user %R (at 0 -1.25 90) (layer F.Fab)
+    (fp_text user %R (at 0 -1.25 90) (layer F.SilkS)
       (effects (font (size 1 1) (thickness 0.15)))
     )
@@
   (module EM78P153S:ultrasonic_speaker (layer F.Cu)
     (at 102.87 104.14 90)
-    (fp_text reference LS1 (at 0 0.5 90) (layer F.SilkS)
-      (effects (font (size 1 1) (thickness 0.15)))
-    )
-    (fp_text value Speaker (at 0 -0.5 90) (layer F.Fab)
+    (fp_text reference LS1 (at 0.127 6.2865 90) (layer F.SilkS)
+      (effects (font (size 1 1) (thickness 0.15)))
+    )
+    (fp_text value Speaker (at 0.0254 4.8133 90) (layer F.SilkS)
       (effects (font (size 1 1) (thickness 0.15)))
     )
@@
   (module EM78P153S:ultrasonic_speaker (layer F.Cu)
     (at 191.77 104.14 90)
-    (fp_text reference LS2 (at 0 0.5 90) (layer F.SilkS)
-      (effects (font (size 1 1) (thickness 0.15)))
-    )
-    (fp_text value Speaker (at 0 -0.5 90) (layer F.Fab)
+    (fp_text reference LS2 (at 0.127 5.8801 90) (layer F.SilkS)
+      (effects (font (size 1 1) (thickness 0.15)))
+    )
+    (fp_text value Speaker (at 0.127 4.3688 90) (layer F.Fab) hide
       (effects (font (size 1 1) (thickness 0.15)))
     )
@@
     (tags "resistor 0603")
     (attr smd)
-    (fp_text reference R2 (at 0 -1.45) (layer F.SilkS)
+    (fp_text reference R2 (at -1.3462 -1.3462) (layer F.SilkS)
       (effects (font (size 1 1) (thickness 0.15)))
     )
@@
       (effects (font (size 1 1) (thickness 0.15)))
     )
-    (fp_text value LM324 (at 0 -0.5 90) (layer F.Fab)
+    (fp_text value LM324 (at 0.0254 -0.8636 90) (layer F.SilkS)
       (effects (font (size 1 1) (thickness 0.15)))
     )
@@
       (effects (font (size 1 1) (thickness 0.15)))
     )
-    (fp_text value EM78P153S (at 0 -0.5 90) (layer F.Fab)
+    (fp_text value EM78P153S (at -1.1938 -0.7493 90) (layer F.SilkS)
       (effects (font (size 1 1) (thickness 0.15)))
     )
@@
       (effects (font (size 1 1) (thickness 0.15)))
     )
-    (fp_text value MAX232A (at 0 -0.5 180) (layer F.Fab)
+    (fp_text value MAX232A (at -0.6731 -0.8763 180) (layer F.SilkS)
       (effects (font (size 1 1) (thickness 0.15)))
     )
@@
     (tags "mounting hole 3mm no annular")
     (attr virtual)
-    (fp_text reference REF** (at 0 -4) (layer F.SilkS)
+    (fp_text reference REF** (at -0.2921 -6.9596) (layer F.SilkS) hide
       (effects (font (size 1 1) (thickness 0.15)))
     )
@@
     (tags "mounting hole 3mm no annular")
     (attr virtual)
-    (fp_text reference REF** (at 0 -4) (layer F.SilkS)
+    (fp_text reference REF** (at 0 -4) (layer F.SilkS) hide
       (effects (font (size 1 1) (thickness 0.15)))
     )
@@
     (tags "mounting hole 3mm no annular")
     (attr virtual)
-    (fp_text reference REF** (at 0 -4) (layer F.SilkS)
+    (fp_text reference REF** (at 0 -4) (layer F.SilkS) hide
       (effects (font (size 1 1) (thickness 0.15)))
     )
@@
     (pad 1 np_thru_hole circle (at 0 0) (size 3 3) (drill 3) (layers *.Cu *.Mask))
   )
-  (gr_text Vcc (at 147.32 120.7135) (layer F.Cu)
+  (gr_text V0.1 (at 171.0817 86.7283) (layer F.SilkS)
     (effects (font (size 1.5 1.5) (thickness 0.3)))
   )
-  (gr_text Trig (at 151.9428 117.3988) (layer F.Cu)
+  (gr_text Vcc (at 149.5679 117.6655) (layer F.SilkS)
+    (effects (font (size 1.5 1.5) (thickness 0.3)))
+  )
+  (gr_text Trig (at 153.5684 118.2497) (layer F.SilkS)
     (effects (font (size 1 1) (thickness 0.2)))
   )
-  (gr_text Echo (at 157.7467 117.5004) (layer F.Cu)
+  (gr_text Echo (at 156.9847 118.1354) (layer F.SilkS)
     (effects (font (size 1 1) (thickness 0.2)))
   )
-  (gr_text GND (at 163.1188 120.8659) (layer F.Cu)
+  (gr_text GND (at 161.5694 117.7798) (layer F.SilkS)
     (effects (font (size 1.5 1.5) (thickness 0.3)))
   )
